Commit message: fixed ros2 control issues

File: src/rbcar_model/robots/rbcar2.urdf.xacro (robot description, xacro)
@@ -9,8 +9,7 @@
 	<xacro:include filename="$(find rbcar_model)/urdf/wheels/suspension_wheel_v3.urdf.xacro" />
 	<!-- Import all available sensors -->
-	<!--
 	<xacro:include filename="$(find robotnik_sensors)/urdf/all_sensors.urdf.xacro" />
+	<!-- <xacro:include filename="$(find robotnik_sensors_gazebo)/urdf/default.urdf.xacro" /> -->
   	<xacro:include filename="$(find robotnik_sensors)/urdf/utils/inertia.urdf.xacro" />
-	-->
 	<!-- ***************** -->
 	<!-- Global parameters -->
@@ -43,25 +42,27 @@
 		lr_reflect="-1" fr_reflect="-1" parent="$(arg prefix)base_link" />
 	<!-- Sensors -->
-	<!--
-	<xacro:sensor_rslidar_16 prefix="$(arg prefix)top_3d_laser" parent="$(arg prefix)base_link"
-	gpu="$(arg gpu)">
+	<!-- Setting gpu to false because the plugin fails -->
+	<!-- <xacro:sensor_rslidar_16 prefix="$(arg prefix)top_3d_laser"  parent="$(arg prefix)base_link"
+	gpu="false">
 	  <origin xyz="1.163 0.0 1.602" rpy="0 0.2637 0"/>
-	</xacro:sensor_rslidar_16>
+	</xacro:sensor_rslidar_16> -->
+	<!-- <xacro:sensor_robosense_helios_16p frame_prefix="$(arg prefix)front_laser" simulation="true" parent="$(arg prefix)base_link"
+	topic_prefix="top_3d_lidar" gpu="$(arg gpu)">
+		<origin xyz="2.101 0 0.206" rpy="0 0 0"/>
+	</xacro:sensor_robosense_helios_16p> -->
 	<xacro:sensor_imu_hector prefix="$(arg prefix)imu" parent="$(arg prefix)base_link">
 		<origin xyz="0.319 0.018 0.676" rpy="0 0 0"/>
 	</xacro:sensor_imu_hector>
-	<xacro:sensor_sick_outdoorscan3 prefix="$(arg prefix)front_laser" parent="$(arg prefix)base_link"
-	prefix_topic="front_laser" min_angle="-1.5" max_angle="1.5" gpu="$(arg gpu)">
+	<xacro:sensor_sick_outdoorscan3 simulation="true" frame_prefix="$(arg prefix)front_laser" parent="$(arg prefix)base_link"
+	topic_prefix="front_laser" gpu="$(arg gpu)">
 		<origin xyz="2.101 0 0.206" rpy="0 0 0"/>
 	</xacro:sensor_sick_outdoorscan3>
-	<xacro:sensor_hokuyo_utm30lx prefix="$(arg prefix)rear_laser" parent="$(arg prefix)base_link"
-	gpu="$(arg gpu)" prefix_topic="rear_laser">
+	<xacro:sensor_hokuyo_utm30lx simulation="true" frame_prefix="$(arg prefix)rear_laser" parent="$(arg prefix)base_link"
+	gpu="$(arg gpu)" topic_prefix="rear_laser">
       		<origin xyz="-0.42925 0.0 0.24674" rpy="0 0 ${PI}"/>
   	</xacro:sensor_hokuyo_utm30lx>
-	<xacro:sensor_gps prefix="$(arg prefix)gps" parent="$(arg prefix)base_link" gps_latitude="$(arg
-	gps_latitude)" gps_longitude="$(arg gps_longitude)">
+	<xacro:sensor_gps node_namespace="rbcar" simulation="true" frame_prefix="$(arg prefix)gps" parent="$(arg prefix)base_link" >
 		<origin xyz="0.491 0 1.503" rpy="0 0 0"/>
 	</xacro:sensor_gps>
-	-->
 	<!-- Gazebo plugins -->
 	<!--

File: src/rbcar_model/urdf/bases/rbcar_base.gazebo.xacro (robot description, xacro)
@@ -3,10 +3,24 @@
   <!-- ros control plugin -->
   <xacro:macro name="ros_control">
+      <gazebo>
+        <plugin filename="libgazebo_ros2_control.so" name="gazebo_ros2_control">
+            <robot_param>robot_description</robot_param>
+            <robot_param_node>robot_state_publisher</robot_param_node>
+            <parameters>$(find rbcar_model)/config/rbcar_controllers.yaml</parameters>
+            <ros>
+                <namespace></namespace>
+                <remapping>ackermann_steering_controller/reference_unstamped:=cmd_vel</remapping>
+                <remapping>ackermann_steering_controller/odometry:=odom</remapping>
+                <remapping>ackermann_steering_controller/tf_odometry:=tf</remapping>
+                <robot_base_frame>base_link</robot_base_frame>
+            </ros>
+        </plugin>
+    </gazebo>
+<!--
     <gazebo>
-      <!-- ROS 2 control plugin -->
       <plugin name='gazebo_ros2_control' filename='libgazebo_ros2_control.so'>
         <parameters>$(find rbcar_model)/config/rbcar_controllers.yaml</parameters>
       </plugin>
-    </gazebo>
+    </gazebo> -->
   </xacro:macro>
   <gazebo reference="base_footprint">

File: src/rbcar_model/urdf/bases/rbcar_base.urdf.xacro (robot description, xacro)
@@ -18,4 +18,9 @@
         </visual>
       </link>
+    <!-- <joint name="world_to_base" type="fixed">
+        <parent link="world"/>
+        <child link="${prefix}base_footprint"/>
+        <origin xyz="0 0 0" rpy="0 0 0"/>
+    </joint> -->
       <joint name="${prefix}base_footprint_joint" type="fixed">
         <origin xyz="0 0 ${clearance}" rpy="0 0 0" />
@@ -62,6 +67,6 @@
       <joint name="${prefix}left_steering_joint">
         <command_interface name="position">
-          <param name="min">-0.6</param>
-          <param name="max">0.785398163</param>
+          <param name="min">${-PI/4}</param>
+          <param name="max">${PI/4}</param>
         </command_interface>
         <state_interface name="position"/>
@@ -70,6 +75,6 @@
       <joint name="${prefix}right_steering_joint">
         <command_interface name="position">
-          <param name="min">-0.785398163</param>
-          <param name="max">0.6</param>
+          <param name="min">${-PI/4}</param>
+          <param name="max">${PI/4}</param>
         </command_interface>
         <state_interface name="position"/>
@@ -89,10 +94,10 @@
       <!-- Rear wheel joints -->
       <joint name="${prefix}left_rear_axle">
-        <!-- <command_interface name="velocity"/> -->
+        <command_interface name="velocity"/>
         <state_interface name="position"/>
         <state_interface name="velocity"/>
       </joint>
       <joint name="${prefix}right_rear_axle">
-        <!-- <command_interface name="velocity"/> -->
+        <command_interface name="velocity"/>
         <state_interface name="position"/>
         <state_interface name="velocity"/>

Commit message: working slam

File: src/rbcar_model/robots/rbcar2.urdf.xacro (robot description, xacro)
@@ -51,7 +51,20 @@
 		<origin xyz="2.101 0 0.206" rpy="0 0 0"/>
 	</xacro:sensor_robosense_helios_16p> -->
-	<xacro:sensor_imu_hector prefix="$(arg prefix)imu" parent="$(arg prefix)base_link">
+	<!-- Comment out existing IMU -->
+	<!-- <xacro:sensor_imu_hector prefix="$(arg prefix)imu" parent="$(arg prefix)base_link">
 		<origin xyz="0.319 0.018 0.676" rpy="0 0 0"/>
-	</xacro:sensor_imu_hector>
+	</xacro:sensor_imu_hector> -->
+	<!-- Add myahrs IMU with correct frame prefix -->
+	    <!-- <xacro:sensor_myahrs frame_prefix="$(arg prefix)imu_" node_namespace="" topic_prefix="imu/" parent="$(arg prefix)base_link" simulation="true" node_name="imu" >
+      <origin xyz="0.319 0.018 0.676" rpy="0 0 0"/> -->
+	<xacro:sensor_myahrs
+		frame_prefix="$(arg prefix)imu_"
+		parent="$(arg prefix)base_link"
+		simulation="true"
+		node_name="imu"
+		node_namespace=""
+		topic_prefix="imu/">
+		<origin xyz="0.319 0.018 0.676" rpy="0 0 0"/>
+	</xacro:sensor_myahrs>
 	<xacro:sensor_sick_outdoorscan3 simulation="true" frame_prefix="$(arg prefix)front_laser" parent="$(arg prefix)base_link"
 	topic_prefix="front_laser" gpu="$(arg gpu)">

Commit message: latest

File: src/rbcar_model/robots/rbcar2.urdf.xacro (robot description, xacro)
@@ -46,4 +46,5 @@
 	gpu="false">
 	  <origin xyz="1.163 0.0 1.602" rpy="0 0.2637 0"/>
+	  <!-- <origin xyz="0.0 0.0 0.0" rpy="0 0 0"/> -->
 	</xacro:sensor_rslidar_16>
 	<!-- <xacro:sensor_robosense_helios_16p frame_prefix="$(arg prefix)front_laser" simulation="true" parent="$(arg prefix)base_link"

File: src/rbcar_model/urdf/bases/rbcar_base.urdf.xacro (robot description, xacro)
@@ -14,4 +14,5 @@
           <origin xyz="0 0 0" rpy="0 0 0" />
           <geometry>
+            <!-- <box size="0.01 0.01 0.01" /> -->
             <box size="0.001 0.001 0.001" />
           </geometry>
@@ -41,4 +42,5 @@
           <geometry>
             <mesh filename="package://rbcar_model/meshes/bases/rbcar_chassis_hq.stl"/>
+            <!-- <box size="0.01 0.01 0.01"/> -->
           </geometry>
         </xacro:if>
@@ -46,4 +48,5 @@
           <geometry>
             <mesh filename="package://rbcar_model/meshes/bases/rbcar_chassis.stl"/>
+            <!-- <box size="0.01 0.01 0.01"/> -->
           </geometry>
         </xacro:unless>
@@ -56,4 +59,5 @@
         <geometry>
           <mesh filename="package://rbcar_model/meshes/bases/rbcar_chassis.stl"/>
+          <!-- <box size="0.01 0.01 0.01"/> -->
         </geometry>
       </collision>
@@ -76,5 +80,5 @@
         <command_interface name="position">
           <param name="min">${-PI/4}</param>
-          <param name="max">${PI/4}</param>
+          <param name="max">${PI/4}</param .>
         </command_interface>
         <state_interface name="position"/>
